Commit message: Add lidar link to enterprise urdf
A simple box has been added to the urdf model of enterprise.  This will
allow gmapping to be used in the future after joint_state_publisher has
been implemented.

File: mst_control/urdf/robots/Enterprise2.URDF (robot description, URDF)
Before this commit: robot Enterprise2, 2 links, 1 joints
Links:
- added link lidar_link, mass 1; visual box size=.1 .1 .1
Joints:
- added joint lidar_link: type fixed, parent base_link, child lidar_link, origin xyz=.1 0 .285 rpy=0 0 0, axis 0 0 0

Commit message: Add gmapping to the code and launch file
Gmapping and the lidar should be integrated into the launch file now.
You may need to install gmapping to run the code, this can be installed
with "sudo apt-get install ros-indigo-gmapping".

File: mst_control/urdf/robots/Enterprise2.URDF (robot description, URDF)
Before this commit: robot Enterprise2, 3 links, 2 joints
Links:
- removed link lidar_link
- added link laser, mass 1; visual box size=.1 .1 .1
Joints:
- removed joint lidar_link
- added joint laser: type fixed, parent base_link, child laser, origin xyz=.1 0 .285 rpy=0 0 0, axis 0 0 0
