Commit message: Change name of mst_control to control
The mst_ prefix is unnecessary and has been removed from the control
package.  The code has been updated to reflect this change and mst_
should not be used as a prefix in any new packages.

File: control/urdf/robots/Enterprise2.URDF (robot description, URDF)
Before this commit: robot Enterprise2, 3 links, 2 joints
Links:
- link Camera: geometry collision mesh filename=package://control/urdf/meshes/Camera.STL; visual mesh filename=package://control/urdf/meshes/Camera.STL
- link base_link: geometry collision mesh filename=package://control/urdf/meshes/base_link.STL; visual mesh filename=package://control/urdf/meshes/base_link.STL
